File: Sweep v2.2/my_sweepv2.kicad_pcb (KiCad board)
At the start: 2 copper layers, 219.1 x 86 mm, 47 parts, among them J1 AudioJack4dpb, J2 AudioJack4dpb, SW10 SW_Push, SW11 SW_Push, SW11_r1 SW_Push, SW12 SW_Push, SW12_r1 SW_Push, SW13_r1 SW_Push, SW14 SW_Push, SW15 SW_Push, SW15_r1 SW_Push, SW16 SW_Push, SW16_r1 SW_Push, SW17 SW_Push, SW17_r1 SW_Push, SW18 SW_Push, SW18_r1 SW_Push, SW2 SW_Push, SW20 SW_Push, SW20_r1 SW_Push, SW21 SW_Push, SW21_r1 SW_Push, SW2_r1 SW_Push, SW3 SW_Push, SW3_r1 SW_Push, SW4 SW_Push, SW4_r1 SW_Push, SW5 SW_Push, SW5_r1 SW_Push, SW6 SW_Push, SW6_r1 SW_Push, SW7_r1 SW_Push, SW8 SW_Push, SW8_r1 SW_Push, SW9 SW_Push, SW9_r1 SW_Push, U1 ProMicro-kbd, U2 ProMicro-kbd

Commit message: Removed files I wasnt using and modified the fill of both v2.2 and half
Parts:
- added mouse-bite-2mm-slot: VAL**, Duckyb-Parts:mouse-bite-5mm-slot-with-space-for-track, F.Cu at (130.4, 50.3)
- moved mouse-bite-2mm-slot 1.09 mm to (130.3, 74.1)
Other:
- outline, holes or cut-outs redrawn
- board text removed: "Sweep is based on the Ferris."
- board text removed: "Sweep v 2.2"
