File: sweep_v2.2/my_sweepv2.kicad_pcb (KiCad board)
At the start: 2 copper layers, 219.1 x 86 mm, 48 parts, among them J1 AudioJack4dpb, J2 AudioJack4dpb, SW10 SW_Push, SW11 SW_Push, SW11_r1 SW_Push, SW12 SW_Push, SW12_r1 SW_Push, SW13_r1 SW_Push, SW14 SW_Push, SW15 SW_Push, SW15_r1 SW_Push, SW16 SW_Push, SW16_r1 SW_Push, SW17 SW_Push, SW17_r1 SW_Push, SW18 SW_Push, SW18_r1 SW_Push, SW2 SW_Push, SW20 SW_Push, SW20_r1 SW_Push, SW21 SW_Push, SW21_r1 SW_Push, SW2_r1 SW_Push, SW3 SW_Push, SW3_r1 SW_Push, SW4 SW_Push, SW4_r1 SW_Push, SW5 SW_Push, SW5_r1 SW_Push, SW6 SW_Push, SW6_r1 SW_Push, SW7_r1 SW_Push, SW8 SW_Push, SW8_r1 SW_Push, SW9 SW_Push, SW9_r1 SW_Push, U1 ProMicro-kbd, U2 ProMicro-kbd

Commit message: fixed trace outside of pcb, started making case
Routing:
- net Switch11_r: track 100.0 -> 81.5 mm
- net Switch12_r: track 71.8 -> 54.3 mm
Changed lines of the file:
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@@
 	)
 	(gr_line
+		(start 85.598 68.072)
+		(end 100.482351 68.060029)
+		(stroke
+			(width 0.2)
+			(type default)
+		)
+		(layer "F.Cu")
+		(net 30)
+	)
+	(gr_line
+		(start 100.482351 68.060029)
+		(end 100.487271 76.82399)
+		(stroke
+			(width 0.2)
+			(type default)
+		)
+		(layer "F.Cu")
+		(net 30)
+	)
+	(gr_line
 		(start 143.775453 89.282)
 		(end 143.724897 77.154637)
@@
 	)
 	(gr_line
+		(start 99.391815 68.588976)
+		(end 99.40587 77.294974)
+		(stroke
+			(width 0.2)
+			(type default)
+		)
+		(layer "F.Cu")
+		(net 31)
+	)
+	(gr_line
 		(start 143.724897 77.154637)
 		(end 156 77.154637)
@@
 		(net 16)
 	)
+	(gr_line
+		(start 85.46959 68.58)
+		(end 99.391815 68.588976)
+		(stroke
+			(width 0.2)
+			(type default)
+		)
+		(layer "F.Cu")
+		(net 31)
+	)
 	(gr_rect
 		(start 27.178 50.419)
@@
 	)
 	(segment
-		(start 87.884 70.358)
-		(end 85.598 68.072)
+		(start 112.318334 78.994)
+		(end 108.204 78.994)
 		(width 0.25)
 		(layer "F.Cu")
@@
 	)
 	(segment
-		(start 116.814833 82.016833)
-		(end 116.103167 81.305167)
+		(start 108.204 78.994)
+		(end 104.902 75.692)
 		(width 0.25)
 		(layer "F.Cu")
@@
 	)
 	(segment
-		(start 116.103167 81.305167)
-		(end 116.103167 81.254833)
+		(start 120.65 89.466)
+		(end 116.814833 85.630833)
 		(width 0.25)
 		(layer "F.Cu")
@@
 	)
 	(segment
-		(start 90.80641 70.358)
-		(end 87.884 70.358)
+		(start 85.598 68.072)
+		(end 84.074 68.072)
 		(width 0.25)
 		(layer "F.Cu")
@@
 	)
 	(segment
-		(start 100.965169 76.82399)
-		(end 97.281308 76.82399)
+		(start 116.814833 82.016833)
+		(end 116.103167 81.305167)
 		(width 0.25)
 		(layer "F.Cu")
@@
 	)
 	(segment
-		(start 114.579167 81.254833)
-		(end 112.318334 78.994)
-		(width 0.25)
-		(layer "F.Cu")
-		(net 30)
-	)
-	(segment
-		(start 85.598 68.072)
-		(end 84.074 68.072)
-		(width 0.25)
-		(layer "F.Cu")
-		(net 30)
-	)
-	(segment
-		(start 102.097159 75.692)
-		(end 100.965169 76.82399)
-		(width 0.25)
-		(layer "F.Cu")
-		(net 30)
-	)
-	(segment
 		(start 81.534 70.612)
 		(end 76.71082 70.612)
@@
 	)
 	(segment
-		(start 116.814833 85.630833)
-		(end 116.814833 82.016833)
-		(width 0.25)
-		(layer "F.Cu")
-		(net 30)
-	)
-	(segment
-		(start 91.127659 70.670341)
-		(end 91.118751 70.670341)
-		(width 0.25)
-		(layer "F.Cu")
-		(net 30)
-	)
-	(segment
 		(start 84.074 68.072)
 		(end 81.534 70.612)
@@
 	)
 	(segment
-		(start 112.318334 78.994)
-		(end 108.204 78.994)
+		(start 100.965169 76.82399)
+		(end 100.487271 76.82399)
 		(width 0.25)
 		(layer "F.Cu")
@@
 	)
 	(segment
-		(start 108.204 78.994)
-		(end 104.902 75.692)
+		(start 76.71082 70.612)
+		(end 72.823121 66.724301)
 		(width 0.25)
 		(layer "F.Cu")
@@
 	)
 	(segment
-		(start 120.65 89.466)
-		(end 116.814833 85.630833)
+		(start 116.814833 85.630833)
+		(end 116.814833 82.016833)
 		(width 0.25)
 		(layer "F.Cu")
@@
 	)
 	(segment
-		(start 76.71082 70.612)
-		(end 72.823121 66.724301)
+		(start 72.823121 66.724301)
+		(end 71.804301 66.724301)
 		(width 0.25)
 		(layer "F.Cu")
@@
 	)
 	(segment
-		(start 72.823121 66.724301)
-		(end 71.804301 66.724301)
+		(start 102.097159 75.692)
+		(end 100.965169 76.82399)
 		(width 0.25)
 		(layer "F.Cu")
@@
 	)
 	(segment
-		(start 97.281308 76.82399)
-		(end 91.127659 70.670341)
+		(start 116.103167 81.305167)
+		(end 116.103167 81.254833)
 		(width 0.25)
 		(layer "F.Cu")
@@
 	)
 	(segment
-		(start 104.902 75.692)
-		(end 102.097159 75.692)
+		(start 114.579167 81.254833)
+		(end 112.318334 78.994)
 		(width 0.25)
 		(layer "F.Cu")
@@
 	)
 	(segment
-		(start 91.118751 70.670341)
-		(end 90.80641 70.358)
+		(start 104.902 75.692)
+		(end 102.097159 75.692)
 		(width 0.25)
 		(layer "F.Cu")
@@
 	)
 	(segment
-		(start 97.086 77.274)
-		(end 102.616 77.274)
-		(width 0.25)
-		(layer "F.Cu")
-		(net 31)
-	)
-	(segment
-		(start 87.75559 70.866)
-		(end 90.678 70.866)
-		(width 0.25)
-		(layer "F.Cu")
-		(net 31)
-	)
-	(segment
 		(start 84.328 68.58)
 		(end 85.46959 68.58)
@@
 	)
 	(segment
-		(start 85.46959 68.58)
-		(end 87.75559 70.866)
+		(start 76.58241 71.12)
+		(end 81.788 71.12)
 		(width 0.25)
 		(layer "F.Cu")
@@
 	)
 	(segment
-		(start 76.58241 71.12)
-		(end 81.788 71.12)
+		(start 60.0659 66.29031)
+		(end 60.841689 67.066099)
 		(width 0.25)
 		(layer "F.Cu")
@@
 	)
 	(segment
-		(start 60.0659 66.29031)
-		(end 60.841689 67.066099)
+		(start 81.788 71.12)
+		(end 84.328 68.58)
 		(width 0.25)
 		(layer "F.Cu")
@@
 	)
 	(segment
-		(start 90.678 70.866)
-		(end 97.086 77.274)
+		(start 60.841689 67.066099)
+		(end 60.841689 67.174311)
 		(width 0.25)
 		(layer "F.Cu")
@@
 	)
 	(segment
-		(start 81.788 71.12)
-		(end 84.328 68.58)
+		(start 99.40587 77.294974)
+		(end 99.426844 77.274)
 		(width 0.25)
 		(layer "F.Cu")
@@
 	)
 	(segment
-		(start 60.841689 67.066099)
-		(end 60.841689 67.174311)
+		(start 99.426844 77.274)
+		(end 102.616 77.274)
 		(width 0.25)
 		(layer "F.Cu")
